File: wall-e.sch (EAGLE design)
At the start: 71 parts, among them IC1 VREG-TS1117CW-3V3, T1 BC847, U1 TSM2306CX, U2 TSM2306CX, U3 TSM2306CX, U4 TSM2306CX, U5 TSM2306CX, U6 TSM2306CX, U7 TSM2306CX, U8 LM293AD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

Commit message: Routing
Connections:
- net BUTTON1: now also U$1.PA1; no longer U$1.PA0
- net BUTTON2: now also U$1.PA0; no longer U$1.PA1
- net JACK: now also U$1.PA5; no longer U$1.PA4
- net N$7: now also PNEUMATIC-6.1; no longer PNEUMATIC-5.1
- net VALVE1: now also U$1.PB2; no longer U$1.PA5
- net VALVE2: now also U$1.PB1; no longer U$1.PB0
- net VALVE3: now also U$1.PB0; no longer U$1.PB1
- net VALVE4: now also U$1.PA4; no longer U$1.PB2
Changed lines of the file:
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@@
 <instance part="GND8" gate="1" x="27.94" y="38.1"/>
 <instance part="P+3" gate="1" x="266.7" y="35.56"/>
-<instance part="P+7" gate="1" x="337.82" y="55.88"/>
+<instance part="P+7" gate="1" x="337.82" y="50.8"/>
 <instance part="R2" gate="G$1" x="147.32" y="35.56"/>
 <instance part="R3" gate="G$1" x="147.32" y="33.02"/>
@@
 </segment>
 <segment>
-<pinref part="U$1" gate="G$1" pin="PA5"/>
-<wire x1="83.82" y1="78.74" x2="86.36" y2="78.74" width="0.1524" layer="91"/>
-<label x="88.9" y="78.74" size="1.778" layer="95"/>
+<pinref part="U$1" gate="G$1" pin="PB2"/>
+<wire x1="83.82" y1="40.64" x2="86.36" y2="40.64" width="0.1524" layer="91"/>
+<label x="88.9" y="40.64" size="1.778" layer="95"/>
 </segment>
 </net>
 <net name="VALVE2" class="0">
+<segment>
+<pinref part="U1" gate="A" pin="G"/>
+<wire x1="276.86" y1="10.16" x2="274.32" y2="10.16" width="0.1524" layer="91"/>
+<label x="271.78" y="7.62" size="1.778" layer="95"/>
+</segment>
+<segment>
+<pinref part="U$1" gate="G$1" pin="PB1"/>
+<wire x1="83.82" y1="43.18" x2="86.36" y2="43.18" width="0.1524" layer="91"/>
+<label x="88.9" y="43.18" size="1.778" layer="95"/>
+</segment>
+</net>
+<net name="VALVE4" class="0">
+<segment>
+<pinref part="U3" gate="A" pin="G"/>
+<wire x1="317.5" y1="10.16" x2="314.96" y2="10.16" width="0.1524" layer="91"/>
+<label x="312.42" y="7.62" size="1.778" layer="95"/>
+</segment>
+<segment>
+<pinref part="U$1" gate="G$1" pin="PA4"/>
+<wire x1="86.36" y1="81.28" x2="83.82" y2="81.28" width="0.1524" layer="91"/>
+<label x="88.9" y="81.28" size="1.778" layer="95"/>
+</segment>
+</net>
+<net name="VALVE3" class="0">
+<segment>
+<pinref part="U2" gate="A" pin="G"/>
+<wire x1="297.18" y1="10.16" x2="294.64" y2="10.16" width="0.1524" layer="91"/>
+<label x="292.1" y="7.62" size="1.778" layer="95"/>
+</segment>
 <segment>
 <pinref part="U$1" gate="G$1" pin="PB0"/>
 <wire x1="83.82" y1="45.72" x2="86.36" y2="45.72" width="0.1524" layer="91"/>
 <label x="88.9" y="45.72" size="1.778" layer="95"/>
-</segment>
-<segment>
-<pinref part="U1" gate="A" pin="G"/>
-<wire x1="276.86" y1="10.16" x2="274.32" y2="10.16" width="0.1524" layer="91"/>
-<label x="271.78" y="7.62" size="1.778" layer="95"/>
-</segment>
-</net>
-<net name="VALVE4" class="0">
-<segment>
-<pinref part="U$1" gate="G$1" pin="PB2"/>
-<wire x1="83.82" y1="40.64" x2="86.36" y2="40.64" width="0.1524" layer="91"/>
-<label x="88.9" y="40.64" size="1.778" layer="95"/>
-</segment>
-<segment>
-<pinref part="U3" gate="A" pin="G"/>
-<wire x1="317.5" y1="10.16" x2="314.96" y2="10.16" width="0.1524" layer="91"/>
-<label x="312.42" y="7.62" size="1.778" layer="95"/>
-</segment>
-</net>
-<net name="VALVE3" class="0">
-<segment>
-<pinref part="U$1" gate="G$1" pin="PB1"/>
-<wire x1="83.82" y1="43.18" x2="86.36" y2="43.18" width="0.1524" layer="91"/>
-<label x="88.9" y="43.18" size="1.778" layer="95"/>
-</segment>
-<segment>
-<pinref part="U2" gate="A" pin="G"/>
-<wire x1="297.18" y1="10.16" x2="294.64" y2="10.16" width="0.1524" layer="91"/>
-<label x="292.1" y="7.62" size="1.778" layer="95"/>
 </segment>
 </net>
@@
 <pinref part="PNEUMATIC" gate="-8" pin="1"/>
 <pinref part="P+7" gate="1" pin="+12V"/>
-<wire x1="342.9" y1="53.34" x2="337.82" y2="53.34" width="0.1524" layer="91"/>
+<wire x1="342.9" y1="53.34" x2="337.82" y2="48.26" width="0.1524" layer="91"/>
 </segment>
 <segment>
@@
 <net name="N$7" class="0">
 <segment>
-<wire x1="327.66" y1="17.78" x2="327.66" y2="60.96" width="0.1524" layer="91"/>
-<pinref part="PNEUMATIC" gate="-5" pin="1"/>
-<wire x1="327.66" y1="60.96" x2="342.9" y2="60.96" width="0.1524" layer="91"/>
+<wire x1="327.66" y1="17.78" x2="327.66" y2="58.42" width="0.1524" layer="91"/>
 <pinref part="U3" gate="A" pin="D"/>
 <pinref part="D3" gate="G$1" pin="A"/>
@@
 <wire x1="320.04" y1="17.78" x2="327.66" y2="17.78" width="0.1524" layer="91"/>
 <junction x="327.66" y="17.78"/>
+<pinref part="PNEUMATIC" gate="-6" pin="1"/>
+<wire x1="342.9" y1="58.42" x2="327.66" y2="58.42" width="0.1524" layer="91"/>
 </segment>
 </net>
@@
 </segment>
 <segment>
-<pinref part="U$1" gate="G$1" pin="PA4"/>
-<wire x1="86.36" y1="81.28" x2="83.82" y2="81.28" width="0.1524" layer="91"/>
-<label x="88.9" y="81.28" size="1.778" layer="95"/>
+<pinref part="U$1" gate="G$1" pin="PA5"/>
+<wire x1="83.82" y1="78.74" x2="86.36" y2="78.74" width="0.1524" layer="91"/>
+<label x="88.9" y="78.74" size="1.778" layer="95"/>
 </segment>
 </net>
@@
 <wire x1="154.94" y1="48.26" x2="152.4" y2="48.26" width="0.1524" layer="91"/>
 <label x="139.7" y="48.26" size="1.778" layer="95"/>
+</segment>
+<segment>
+<pinref part="U$1" gate="G$1" pin="PA1"/>
+<wire x1="83.82" y1="88.9" x2="86.36" y2="88.9" width="0.1524" layer="91"/>
+<label x="88.9" y="88.9" size="1.778" layer="95"/>
+</segment>
+</net>
+<net name="BUTTON2" class="0">
+<segment>
+<pinref part="TOIT" gate="-5" pin="1"/>
+<wire x1="154.94" y1="45.72" x2="152.4" y2="45.72" width="0.1524" layer="91"/>
+<label x="139.7" y="45.72" size="1.778" layer="95"/>
 </segment>
 <segment>
@@
 </segment>
 </net>
-<net name="BUTTON2" class="0">
-<segment>
-<pinref part="TOIT" gate="-5" pin="1"/>
-<wire x1="154.94" y1="45.72" x2="152.4" y2="45.72" width="0.1524" layer="91"/>
-<label x="139.7" y="45.72" size="1.778" layer="95"/>
-</segment>
-<segment>
-<pinref part="U$1" gate="G$1" pin="PA1"/>
-<wire x1="83.82" y1="88.9" x2="86.36" y2="88.9" width="0.1524" layer="91"/>
-<label x="88.9" y="88.9" size="1.778" layer="95"/>
-</segment>
-</net>
 <net name="BUTTON3" class="0">
 <segment>
@@
 <net name="LED2" class="0">
 <segment>
+<pinref part="R3" gate="G$1" pin="1"/>
+<wire x1="142.24" y1="33.02" x2="139.7" y2="33.02" width="0.1524" layer="91"/>
+<label x="132.08" y="33.02" size="1.778" layer="95"/>
+</segment>
+<segment>
 <pinref part="U$1" gate="G$1" pin="PA7"/>
 <wire x1="83.82" y1="73.66" x2="86.36" y2="73.66" width="0.1524" layer="91"/>
 <label x="88.9" y="73.66" size="1.778" layer="95"/>
-</segment>
-<segment>
-<pinref part="R3" gate="G$1" pin="1"/>
-<wire x1="142.24" y1="33.02" x2="139.7" y2="33.02" width="0.1524" layer="91"/>
-<label x="132.08" y="33.02" size="1.778" layer="95"/>
 </segment>
 </net>
@@
 <wire x1="236.22" y1="17.78" x2="236.22" y2="20.32" width="0.1524" layer="91"/>
 <wire x1="236.22" y1="20.32" x2="236.22" y2="22.86" width="0.1524" layer="91"/>
-<wire x1="243.84" y1="20.32" x2="243.84" y2="58.42" width="0.1524" layer="91"/>
-<wire x1="243.84" y1="58.42" x2="340.36" y2="58.42" width="0.1524" layer="91"/>
-<wire x1="340.36" y1="58.42" x2="340.36" y2="55.88" width="0.1524" layer="91"/>
+<wire x1="243.84" y1="20.32" x2="243.84" y2="55.88" width="0.1524" layer="91"/>
+<wire x1="243.84" y1="55.88" x2="342.9" y2="55.88" width="0.1524" layer="91"/>
 <pinref part="PNEUMATIC" gate="-7" pin="1"/>
-<wire x1="340.36" y1="55.88" x2="342.9" y2="55.88" width="0.1524" layer="91"/>
 <wire x1="236.22" y1="20.32" x2="243.84" y2="20.32" width="0.1524" layer="91"/>
 <junction x="236.22" y="20.32"/>

Commit message: fixed board
Parts:
- C14: value 10nF -> 100nF
- C3: value 1uF -> 4.7uF
- C9: device resistor:CPOL-USE2.5-7 -> resistor:CPOL-USE3.5-8
Changed lines of the file:
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@@
 <?xml version="1.0" encoding="utf-8"?>
 <!DOCTYPE eagle SYSTEM "eagle.dtd">
-<eagle version="8.0.2">
+<eagle version="8.1.0">
 <drawing>
 <settings>
@@
 <part name="R8" library="resistor" deviceset="R-US_" device="R0805" value="360R"/>
 <part name="R9" library="resistor" deviceset="R-US_" device="R0805" value="22K"/>
-<part name="C9" library="resistor" deviceset="CPOL-US" device="E2.5-7" value="220uF"/>
+<part name="C9" library="resistor" deviceset="CPOL-US" device="E3.5-8" value="220uF"/>
 <part name="C10" library="resistor" deviceset="CPOL-US" device="E2.5-7" value="220uF"/>
 <part name="C11" library="resistor" deviceset="C-US" device="C0805" value="100n"/>
@@
 <part name="LED1" library="led" deviceset="LED" device="CHIP-LED0805"/>
 <part name="GND28" library="supply1" deviceset="GND" device=""/>
-<part name="C3" library="rcl" deviceset="C-EU" device="C0805" value="1uF"/>
+<part name="C3" library="rcl" deviceset="C-EU" device="C0805" value="4.7uF"/>
 <part name="+3V16" library="supply1" deviceset="+3V3" device=""/>
 <part name="C1" library="rcl" deviceset="C-EU" device="C0805" value="10uF"/>
 <part name="C2" library="rcl" deviceset="C-EU" device="C0805" value="10uF"/>
-<part name="C14" library="rcl" deviceset="C-EU" device="C0805" value="10nF"/>
+<part name="C14" library="rcl" deviceset="C-EU" device="C0805" value="100nF"/>
 <part name="JP1" library="SparkFun" deviceset="M08" device="LONGPADS"/>
 <part name="JP2" library="SparkFun" deviceset="M08" device="LONGPADS"/>
